File: kicad/pog.kicad_pcb (KiCad board)
At the start: 2 copper layers, 179 parts, among them P1 USB_C_Plug_USB2.0, U1 ATmega32U4-A

Commit message: more traces and git ignore update
Parts:
- removed P1: USB_C_Plug_USB2.0, Connector_USB:USB_C_Receptacle_HRO_TYPE-C-31-M-12
Connections:
- U1 pad 36: unconnected-(U1-PF7-Pad36) -> Row 1
- U1 pad 37: Row 5 -> Row 2
- U1 pad 38: Row 4 -> Row 3
- U1 pad 39: Row 3 -> Row 4
- U1 pad 40: Row 2 -> Row 5
- U1 pad 41: Row 1 -> Row 6
Routing:
- net Row 2: track 382.1 -> 518.5 mm, vias 0 -> 2
- net Row 1: track 594.1 -> 567.9 mm
- net Row 6: track 368.5 -> 393.1 mm

Commit message: schematic done
Parts:
- added C1: 1u, Capacitor_SMD:C_1206_3216Metric, B.Cu at (180.4, 124.4)
- added Ground1: TestPoint, TestPoint:TestPoint_THTPad_2.0x2.0mm_Drill1.0mm, B.Cu at (125.6, 122.0)
- added J1: USB_C_Receptacle, USB_C:USB_C_Receptacle_HRO_TYPE-C-31-M-12, B.Cu at (46.0, 21.0)
- added R1: R, Resistor_SMD:R_1206_3216Metric, B.Cu at (46.1, 116.4)
- added R2: R, Resistor_SMD:R_1206_3216Metric, B.Cu at (42.6, 116.4)
- added R3: 5.1k, Resistor_SMD:R_1206_3216Metric, B.Cu at (54.8, 20.8)
- added R4: 5.1k, Resistor_SMD:R_1206_3216Metric, B.Cu at (54.8, 23.2)
- added R5: 10k, Resistor_SMD:R_1206_3216Metric, B.Cu at (138.1, 120.6)
- added R6: 10k, Resistor_SMD:R_1206_3216Metric, B.Cu at (157.5, 115.5)
- added Reset1: TestPoint, TestPoint:TestPoint_THTPad_2.0x2.0mm_Drill1.0mm, B.Cu at (132.5, 122.0)
- moved D1 15.8 mm to (35.9, 36.6), turned to 180 degrees
- moved D2 15.8 mm to (54.9, 36.6), turned to 180 degrees
- moved D17 12.0 mm to (30.7, 55.7), turned to 180 degrees
- turned MX1 to 180 degrees
- turned MX2 to 180 degrees
Connections:
- MX1 pad 1: Net-(MX1-Pad1) -> Column 1
- MX10 pad 1: Net-(MX10-Pad1) -> Column 10
- MX11 pad 1: Net-(MX11-Pad1) -> Column 11
- MX12 pad 1: Net-(MX12-Pad1) -> Column 12
- MX13 pad 1: Net-(MX13-Pad1) -> Column 13
- MX14 pad 1: Net-(MX14-Pad1) -> Column 14
- MX15 pad 1: Net-(MX15-Pad1) -> Column 15
- MX16 pad 1: unconnected-(MX16-Pad1) -> Column 16
- MX17 pad 1: Net-(MX1-Pad1) -> Column 1
- MX18 pad 1: Net-(MX18-Pad1) -> Column 2
- MX19 pad 1: Net-(MX19-Pad1) -> Column 3
- MX2 pad 1: Net-(MX18-Pad1) -> Column 2
- MX20 pad 1: Net-(MX20-Pad1) -> Column 4
- MX21 pad 1: Net-(MX21-Pad1) -> Column 5
- MX22 pad 1: Net-(MX22-Pad1) -> Column 6
- MX23 pad 1: Net-(MX23-Pad1) -> Column 7
- MX24 pad 1: Net-(MX24-Pad1) -> Column 8
- MX25 pad 1: Net-(MX25-Pad1) -> Column 9
- MX26 pad 1: Net-(MX10-Pad1) -> Column 10
- MX27 pad 1: Net-(MX11-Pad1) -> Column 11
- MX28 pad 1: Net-(MX12-Pad1) -> Column 12
- MX29 pad 1: Net-(MX13-Pad1) -> Column 13
- MX3 pad 1: Net-(MX19-Pad1) -> Column 3
- MX30 pad 1: Net-(MX14-Pad1) -> Column 15
- MX31 pad 1: Net-(MX15-Pad1) -> Column 16
- MX32 pad 1: Net-(MX1-Pad1) -> Column 1
- MX33 pad 1: Net-(MX18-Pad1) -> Column 2
- MX34 pad 1: Net-(MX19-Pad1) -> Column 3
- MX35 pad 1: Net-(MX20-Pad1) -> Column 4
- MX36 pad 1: Net-(MX21-Pad1) -> Column 5
- MX37 pad 1: Net-(MX22-Pad1) -> Column 6
- MX38 pad 1: Net-(MX23-Pad1) -> Column 7
- MX39 pad 1: Net-(MX24-Pad1) -> Column 8
- MX4 pad 1: Net-(MX20-Pad1) -> Column 4
- MX40 pad 1: Net-(MX25-Pad1) -> Column 9
- MX41 pad 1: Net-(MX10-Pad1) -> Column 10
- MX42 pad 1: Net-(MX11-Pad1) -> Column 11
- MX43 pad 1: Net-(MX12-Pad1) -> Column 12
- MX44 pad 1: Net-(MX13-Pad1) -> Column 13
- MX45 pad 1: Net-(MX14-Pad1) -> Column 15
- MX46 pad 1: Net-(MX15-Pad1) -> Column 16
- MX47 pad 1: Net-(MX1-Pad1) -> Column 1
- MX48 pad 1: Net-(MX18-Pad1) -> Column 2
- MX49 pad 1: Net-(MX19-Pad1) -> Column 3
- MX5 pad 1: Net-(MX21-Pad1) -> Column 5
- MX50 pad 1: Net-(MX20-Pad1) -> Column 4
- MX51 pad 1: Net-(MX21-Pad1) -> Column 5
- MX52 pad 1: Net-(MX22-Pad1) -> Column 6
- MX53 pad 1: Net-(MX23-Pad1) -> Column 7
- MX54 pad 1: Net-(MX24-Pad1) -> Column 8
- MX55 pad 1: Net-(MX25-Pad1) -> Column 9
- MX56 pad 1: Net-(MX10-Pad1) -> Column 10
- MX57 pad 1: Net-(MX11-Pad1) -> Column 11
- MX58 pad 1: Net-(MX12-Pad1) -> Column 12
- MX59 pad 1: Net-(MX13-Pad1) -> Column 13
- MX6 pad 1: Net-(MX22-Pad1) -> Column 6
- MX60 pad 1: Net-(MX15-Pad1) -> Column 16
- MX61 pad 1: Net-(MX1-Pad1) -> Column 1
- MX62 pad 1: Net-(MX18-Pad1) -> Column 2
- MX63 pad 1: Net-(MX19-Pad1) -> Column 3
- MX64 pad 1: Net-(MX20-Pad1) -> Column 4
- MX65 pad 1: Net-(MX21-Pad1) -> Column 5
- MX66 pad 1: Net-(MX22-Pad1) -> Column 6
- MX67 pad 1: Net-(MX23-Pad1) -> Column 7
- MX68 pad 1: Net-(MX24-Pad1) -> Column 8
- MX69 pad 1: Net-(MX25-Pad1) -> Column 9
- MX7 pad 1: Net-(MX23-Pad1) -> Column 7
- MX70 pad 1: Net-(MX10-Pad1) -> Column 10
- MX71 pad 1: Net-(MX11-Pad1) -> Column 11
- MX72 pad 1: Net-(MX12-Pad1) -> Column 12
- MX73 pad 1: Net-(MX13-Pad1) -> Column 13
- MX74 pad 1: Net-(MX14-Pad1) -> Column 15
- MX75 pad 1: Net-(MX15-Pad1) -> Column 16
- MX76 pad 1: Net-(MX1-Pad1) -> Column 1
- MX77 pad 1: Net-(MX18-Pad1) -> Column 2
- MX78 pad 1: Net-(MX19-Pad1) -> Column 3
- MX79 pad 1: Net-(MX20-Pad1) -> Column 4
- MX8 pad 1: Net-(MX24-Pad1) -> Column 8
- MX80 pad 1: Net-(MX21-Pad1) -> Column 7
- MX81 pad 1: Net-(MX22-Pad1) -> Column 10
- MX82 pad 1: Net-(MX23-Pad1) -> Column 11
- MX83 pad 1: Net-(MX24-Pad1) -> Column 12
- MX84 pad 1: Net-(MX25-Pad1) -> Column 13
- MX85 pad 1: Net-(MX10-Pad1) -> Column 14
- MX86 pad 1: Net-(MX14-Pad1) -> Column 15
- MX87 pad 1: Net-(MX15-Pad1) -> Column 16
- MX9 pad 1: Net-(MX25-Pad1) -> Column 9
- U1 pad 1: unconnected-(U1-PE6-Pad1) -> Column 9
- U1 pad 10: unconnected-(U1-PB2-Pad10) -> Column 12
- U1 pad 11: unconnected-(U1-PB3-Pad11) -> Column 13
- U1 pad 13: unconnected-(U1-~{RESET}-Pad13) -> Net-(U1-~{RESET})
- U1 pad 14: Net-(U1-VCC-Pad14) -> VCC
- U1 pad 15: Net-(U1-GND-Pad15) -> GND
- U1 pad 18: unconnected-(U1-PD0-Pad18) -> Column 14
- U1 pad 19: unconnected-(U1-PD1-Pad19) -> Column 15
- U1 pad 2: unconnected-(U1-UVCC-Pad2) -> VCC
- U1 pad 20: unconnected-(U1-PD2-Pad20) -> Column 16
- U1 pad 22: unconnected-(U1-PD5-Pad22) -> Row 6
- U1 pad 23: Net-(U1-GND-Pad15) -> GND
- U1 pad 24: Net-(U1-AVCC-Pad24) -> VCC
- U1 pad 26: unconnected-(U1-PD6-Pad26) -> Column 1
- U1 pad 27: unconnected-(U1-PD7-Pad27) -> Column 2
- U1 pad 28: unconnected-(U1-PB4-Pad28) -> Column 3
- U1 pad 29: unconnected-(U1-PB5-Pad29) -> Column 4
- U1 pad 3: unconnected-(U1-D--Pad3) -> Net-(U1-D-)
- U1 pad 30: unconnected-(U1-PB6-Pad30) -> Column 7
- U1 pad 31: unconnected-(U1-PC6-Pad31) -> Column 5
- U1 pad 32: unconnected-(U1-PC7-Pad32) -> Column 6
- U1 pad 33: unconnected-(U1-~{HWB}/PE2-Pad33) -> Net-(U1-~{HWB}/PE2)
- U1 pad 34: Net-(U1-VCC-Pad14) -> VCC
- U1 pad 35: Net-(U1-GND-Pad15) -> GND
- U1 pad 4: unconnected-(U1-D+-Pad4) -> Net-(U1-D+)
- U1 pad 41: Row 6 -> Column 8
- U1 pad 43: Net-(U1-GND-Pad15) -> GND
- U1 pad 44: Net-(U1-AVCC-Pad24) -> VCC
- U1 pad 5: unconnected-(U1-UGND-Pad5) -> GND
- U1 pad 6: unconnected-(U1-UCAP-Pad6) -> Net-(U1-UCAP)
- U1 pad 7: unconnected-(U1-VBUS-Pad7) -> VCC
- U1 pad 8: unconnected-(U1-PB0-Pad8) -> Column 10
- U1 pad 9: unconnected-(U1-PB1-Pad9) -> Column 11
Routing:
- net Column 16: track 0.00 -> 259.5 mm, vias 0 -> 1
- net Column 15: track 0.00 -> 245.3 mm, vias 0 -> 1
- net Column 1: track 0.00 -> 229.4 mm, vias 0 -> 1
- net Column 14: track 0.00 -> 221.5 mm, vias 0 -> 1
- net Column 2: track 0.00 -> 212.9 mm, vias 0 -> 1
- net Column 13: track 0.00 -> 200.3 mm, vias 0 -> 1
- net Column 3: track 0.00 -> 194.5 mm, vias 0 -> 1
- net Column 12: track 0.00 -> 180.9 mm, vias 0 -> 1
- net Column 4: track 0.00 -> 175.1 mm, vias 0 -> 1
- net Net-(MX24-Pad1): track 168.2 -> 0.00 mm
- net Net-(MX25-Pad1): track 167.9 -> 0.00 mm
- net Net-(MX22-Pad1): track 167.2 -> 0.00 mm
- net Net-(MX10-Pad1): track 167.2 -> 0.00 mm
- net Net-(MX23-Pad1): track 165.7 -> 0.00 mm
- net Column 11: track 0.00 -> 161.9 mm, vias 0 -> 1
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
Commit message: complete basic pcb design
Parts:
- moved C1 166.7 mm to (28.0, 56.9), turned to 0 degrees
- moved U1 138.1 mm to (47.0, 58.7), turned to -45 degrees
- moved Reset1 122.7 mm to (25.0, 62.8), turned to 90 degrees
- moved R5 121.1 mm to (35.1, 56.9), turned to 180 degrees
- moved Ground1 113.8 mm to (25.0, 68.8), turned to 90 degrees
- moved R6 111.0 mm to (53.3, 77.1), turned to 0 degrees
- moved R1 67.0 mm to (39.6, 49.7)
- moved R2 66.7 mm to (42.0, 49.7)
- moved D30 17.0 mm to (291.7, 43.5), turned to -90 degrees
- moved D17 16.4 mm to (29.5, 39.3)
- moved D32 15.7 mm to (40.5, 74.7), turned to 180 degrees
- moved R3 14.3 mm to (40.8, 23.5), turned to 0 degrees
- moved R4 14.3 mm to (40.8, 20.5), turned to 0 degrees
- moved D45 14.1 mm to (293.8, 62.5), turned to -90 degrees
- moved D1 12.7 mm to (48.5, 36.9)
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Connections:
- U1 pad 1: Column 9 -> Column 1
- U1 pad 10: Column 12 -> Column 3
- U1 pad 11: Column 13 -> Column 4
- U1 pad 18: Column 14 -> Column 5
- U1 pad 19: Column 15 -> Column 6
- U1 pad 20: Column 16 -> Column 7
- U1 pad 21: unconnected-(U1-PD3-Pad21) -> Column 8
- U1 pad 22: Row 6 -> Column 9
- U1 pad 25: unconnected-(U1-PD4-Pad25) -> Column 10
- U1 pad 26: Column 1 -> Column 11
- U1 pad 27: Column 2 -> Column 12
- U1 pad 28: Column 3 -> Column 13
- U1 pad 29: Column 4 -> Column 15
- U1 pad 30: Column 7 -> Column 16
- U1 pad 31: Column 5 -> Column 14
- U1 pad 32: Column 6 -> Column 2
- U1 pad 36: Row 1 -> unconnected-(U1-PF7-Pad36)
- U1 pad 37: Row 2 -> unconnected-(U1-PF6-Pad37)
- U1 pad 38: Row 3 -> Row 6
- U1 pad 39: Row 4 -> Row 5
- U1 pad 40: Row 5 -> Row 4
- U1 pad 41: Column 8 -> Row 3
- U1 pad 8: Column 10 -> Row 2
- U1 pad 9: Column 11 -> Row 1
Routing:
- net Row 1: track 463.6 -> 309.8 mm
- net Net-(U1-D+): track 151.8 -> 5.85 mm, vias 2 -> 0
- net Net-(U1-D-): track 149.8 -> 5.94 mm, vias 2 -> 0
- net Row 2: track 437.3 -> 309.8 mm, vias 2 -> 3
- net Row 3: track 435.6 -> 312.8 mm, vias 2 -> 0
- net Column 1: track 229.4 -> 110.7 mm
- net Column 13: track 200.3 -> 317.9 mm, vias 1 -> 0
- net Column 12: track 180.9 -> 298.1 mm, vias 1 -> 0
- net Column 11: track 161.9 -> 278.2 mm, vias 1 -> 0
- net Column 10: track 143.2 -> 258.4 mm, vias 1 -> 0
- net Column 14: track 221.5 -> 334.9 mm
- net Column 16: track 259.5 -> 364.9 mm, vias 1 -> 0
- net Column 9: track 112.1 -> 215.3 mm, vias 1 -> 0
- net Column 15: track 245.3 -> 347.7 mm, vias 1 -> 0
- net Column 2: track 212.9 -> 110.6 mm
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Other:
- board outline added: 304.2 x 115.2 mm

Commit message: pre switch flip
Parts:
- added H1: MountingHole, MountingHole:MountingHole_2.1mm, F.Cu at (60.4, 28.9)
- added H2: MountingHole, MountingHole:MountingHole_2.1mm, F.Cu at (136.4, 28.9)
- added H3: MountingHole, MountingHole:MountingHole_2.1mm, F.Cu at (212.4, 28.9)
- added H4: MountingHole, MountingHole:MountingHole_2.1mm, F.Cu at (288.4, 28.9)
- added H5: MountingHole, MountingHole:MountingHole_2.1mm, F.Cu at (280.9, 66.8)
- added H6: MountingHole, MountingHole:MountingHole_2.1mm, F.Cu at (47.4, 122.9)
- added H7: MountingHole, MountingHole:MountingHole_2.1mm, F.Cu at (212.4, 122.9)
- added H8: MountingHole, MountingHole:MountingHole_2.1mm, F.Cu at (288.4, 122.9)
- moved D2 11.1 mm to (57.4, 36.9), turned to 180 degrees
- moved R3 9.50 mm to (31.3, 23.5)
- moved R4 9.50 mm to (31.3, 20.5)
- moved D77 8.97 mm to (50.4, 114.9), turned to 180 degrees
- moved D7 8.65 mm to (145.0, 32.1), turned to 180 degrees
- moved D3 8.52 mm to (69.1, 32.1), turned to 180 degrees
- moved D84 8.52 mm to (259.6, 127.4), turned to 180 degrees
- moved D11 8.47 mm to (221.6, 32.1), turned to 180 degrees
- moved D15 8.47 mm to (297.8, 32.1), turned to 180 degrees
- moved J1 7.14 mm to (43.2, 20.2)
- turned MX11 to 0 degrees
- turned MX15 to 0 degrees
- turned MX3 to 0 degrees
- turned MX7 to 0 degrees
- turned MX77 to 0 degrees
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Routing:
- net Row 1: track 309.8 -> 372.4 mm
- net Row 6: track 343.7 -> 370.4 mm
- net Column 3: track 129.5 -> 138.6 mm
- net Column 7: track 196.9 -> 205.1 mm
- net Column 15: track 347.7 -> 355.9 mm
- net Column 13: track 317.9 -> 309.7 mm
- net Column 11: track 278.2 -> 286.5 mm
- net Net-(D77-A): track 7.63 -> 0.00 mm
- net Net-(D2-A): track 10.9 -> 4.56 mm
- net Net-(J1-D--PadA7): track 33.7 -> 28.2 mm
- net VCC: track 86.5 -> 81.3 mm
- net Net-(J1-D+-PadA6): track 31.7 -> 28.8 mm
- net Net-(J1-CC2): track 12.0 -> 14.9 mm
- net Net-(J1-CC1): track 9.82 -> 11.8 mm
- net Column 2: track 110.6 -> 108.7 mm
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Other:
- outline, holes or cut-outs redrawn

Commit message: pcb done except for ground
Parts:
- MX1, MX10, MX11, MX12, MX13, MX14, MX15, MX16, MX17, MX18, MX19, MX2, MX20, MX21, MX22, MX23, MX24, MX25, MX26, MX27, MX28, MX29, MX3, MX30, MX31, MX32, MX33, MX34, MX35, MX36, MX37, MX38, MX39, MX4, MX40, MX41, MX42, MX43, MX44, MX45, MX46, MX47, MX48, MX49, MX5, MX50, MX51, MX52, MX53, MX54, MX55, MX56, MX57, MX58, MX59, MX6, MX60, MX61, MX62, MX63, MX64, MX65, MX66, MX67, MX68, MX69, MX7, MX70, MX71, MX72, MX73, MX74, MX75, MX76, MX77, MX78, MX79, MX8, MX80, MX81, MX82, MX83, MX84, MX85, MX86, MX87, MX9: moved to B.Cu
- moved D2 13.1 mm to (53.6, 24.4), turned to -90 degrees
- moved D18 12.0 mm to (60.3, 42.0)
- moved D11 8.24 mm to (218.8, 24.4), turned to -90 degrees
- moved D15 8.24 mm to (295.0, 24.4), turned to -90 degrees
- moved D3 8.19 mm to (66.4, 24.4), turned to -90 degrees
- moved D7 8.10 mm to (142.6, 24.4), turned to -90 degrees
- moved D19 6.55 mm to (66.1, 43.5)
- moved D73 6.25 mm to (268.8, 100.6)
- moved D10 6.25 mm to (199.7, 24.4)
- moved D12 6.25 mm to (237.8, 24.4)
- moved D20 6.25 mm to (85.4, 43.5)
- moved D21 6.25 mm to (104.5, 43.5)
- moved D22 6.25 mm to (123.5, 43.5)
- moved D23 6.25 mm to (142.6, 43.5)
- moved D24 6.25 mm to (161.6, 43.5)
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Routing:
- net Row 1: track 372.4 -> 328.6 mm
- net Column 2: track 108.7 -> 128.1 mm
- net Column 13: track 309.7 -> 326.9 mm
- net Row 2: track 309.8 -> 296.1 mm
- net Column 8: track 196.6 -> 204.3 mm
- net Net-(D2-A): track 4.56 -> 12.3 mm
- net Net-(D77-A): track 0.00 -> 7.69 mm
- net Column 10: track 258.4 -> 266.0 mm
- net Column 9: track 215.3 -> 222.9 mm
- net Column 5: track 140.6 -> 148.2 mm
- net Column 4: track 150.9 -> 158.6 mm
- net Column 16: track 364.9 -> 372.5 mm
- net Column 12: track 298.1 -> 305.8 mm
- net Column 6: track 159.2 -> 166.8 mm
- net Column 1: track 110.7 -> 117.4 mm, vias 1 -> 2
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